File: CAD/Kicad/Kicad.kicad_sch (KiCad schematic)
At the start: 72 parts, among them J1 USB_C_Receptacle_USB2.0_14P, J2 Conn_01x04_Pin, J3 RJ12_Shielded, J4 USB_C_Receptacle_USB2.0_14P, J5 USB_C_Receptacle_USB2.0_14P, J6 Conn_01x24_Pin, U1 ESP8266EX, U2 AMS1117, U3 SST25VF080B-50-4x-S2Ax, U4 FT230XS, U5 ESP32-S3-NEW, U6 FT230XS, U7 AMS1117, U8 SST25VF080B-50-4x-S2Ax, U9 AMS1117, Y1 Crystal_GND24, Y2 Crystal_GND23

Commit message: sensing revisions
Parts:
- removed J3: RJ12_Shielded, symbol Connector:RJ12_Shielded
- added J3: RJ45_Shielded, symbol Connector:RJ45_Shielded
Connections:
- net C_5V: now also J3.3
- net GND: now also J3.1, J3.SH
- net MAIN_BUS_I2C_SCK: now also J3.5
- net MAIN_BUS_I2C_SDA: now also J3.6
- net VCC2: now also J3.4
- new net INT: J3.2
Other:
- note added: "Add warning to NOT connect this to a non Cloudboard board!"
- note added: "RJ45 sensor board connector"
- note removed: "RJ12 sensor board connector"
Changed lines of the file:
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@@
 		)
 	)
-	(text "RJ12 sensor board connector"
+	(text "RJ45 sensor board connector"
 		(exclude_from_sim no)
-		(at 32.766 199.39 0)
+		(at 32.766 195.58 0)
 		(effects
 			(font
@@
 		)
 	)
+	(text "Add warning to NOT connect this to a non Cloudboard board!"
+		(exclude_from_sim no)
+		(at 79.248 202.438 0)
+		(effects
+			(font
+				(size 1.27 1.27)
+			)
+		)
+	)
 	(text "ESP-S3 ANT"
 		(exclude_from_sim no)
@@
 	(wire
 		(pts
+			(xy 43.18 220.98) (xy 50.8 220.98)
+		)
+		(stroke
+			(width 0)
+			(type default)
+		)
+	)
+	(wire
+		(pts
 			(xy 378.46 157.48) (xy 382.27 157.48)
 		)
@@
 		)
 	)
+	(label "INT"
+		(at 50.8 220.98 0)
+		(effects
+			(font
+				(size 1.27 1.27)
+			)
+			(justify left bottom)
+		)
+	)
 	(label "MAIN_BUS_I2C_SCK"
 		(at 196.85 15.24 0)
@@
 	)
 	(symbol
-		(lib_id "Connector:RJ12_Shielded")
-		(at 33.02 218.44 0)
-		(unit 1)
-		(body_style 1)
-		(exclude_from_sim no)
-		(in_bom yes)
-		(on_board yes)
-		(in_pos_files yes)
-		(dnp no)
-		(fields_autoplaced yes)
-		(property "Reference" "J3"
-			(at 33.02 203.2 0)
-			(show_name no)
-			(do_not_autoplace no)
-			(effects
-				(font
-					(size 1.27 1.27)
-				)
-			)
-		)
-		(property "Value" "RJ12_Shielded"
-			(at 33.02 205.74 0)
-			(show_name no)
-			(do_not_autoplace no)
-			(effects
-				(font
-					(size 1.27 1.27)
-				)
-			)
-		)
-		(property "Footprint" ""
-			(at 33.02 217.805 90)
-			(hide yes)
-			(show_name no)
-			(do_not_autoplace no)
-			(effects
-				(font
-					(size 1.27 1.27)
-				)
-			)
-		)
-		(property "Datasheet" ""
-			(at 33.02 217.805 90)
-			(hide yes)
-			(show_name no)
-			(do_not_autoplace no)
-			(effects
-				(font
-					(size 1.27 1.27)
-				)
-			)
-		)
-		(property "Description" "RJ connector, 6P6C (6 positions 6 connected), Shielded"
-			(at 33.02 218.44 0)
-			(hide yes)
-			(show_name no)
-			(do_not_autoplace no)
-			(effects
-				(font
-					(size 1.27 1.27)
-				)
-			)
-		)
-		(pin "6"
-		)
-		(pin "5"
-		)
-		(pin "4"
-		)
-		(pin "3"
-		)
-		(pin "1"
-		)
-		(pin "SH"
-		)
-		(pin "2"
-		)
-		(instances
-			(project "Kicad"
-				(path "/a972b0d3-46a0-4f09-b60b-5ab9fef2950e"
-					(reference "J3")
-					(unit 1)
-				)
-			)
-		)
-	)
-	(symbol
 		(lib_id "Device:C")
 		(at 26.67 31.75 180)
@@
 					(unit 1)
 				)
+			)
+		)
+	)
+	(symbol
+		(lib_id "Connector:RJ45_Shielded")
+		(at 33.02 215.9 0)
+		(unit 1)
+		(body_style 1)
+		(exclude_from_sim no)
+		(in_bom yes)
+		(on_board yes)
+		(in_pos_files yes)
+		(dnp no)
+		(fields_autoplaced yes)
+		(property "Reference" "J3"
+			(at 33.02 198.12 0)
+			(show_name no)
+			(do_not_autoplace no)
+			(effects
+				(font
+					(size 1.27 1.27)
+				)
+			)
+		)
+		(property "Value" "RJ45_Shielded"
+			(at 33.02 200.66 0)
+			(show_name no)
+			(do_not_autoplace no)
+			(effects
+				(font
+					(size 1.27 1.27)
+				)
+			)
+		)
+		(property "Footprint" ""
+			(at 33.02 215.265 90)
+			(hide yes)
+			(show_name no)
+			(do_not_autoplace no)
+			(effects
+				(font
+					(size 1.27 1.27)
+				)
+			)
+		)
+		(property "Datasheet" ""
+			(at 33.02 215.265 90)
+			(hide yes)
+			(show_name no)
+			(do_not_autoplace no)
+			(effects
+				(font
+					(size 1.27 1.27)
+				)
+			)
+		)
+		(property "Description" "RJ connector, 8P8C (8 positions 8 connected), Shielded"
+			(at 33.02 215.9 0)
+			(hide yes)
+			(show_name no)
+			(do_not_autoplace no)
+			(effects
+				(font
+					(size 1.27 1.27)
+				)
+			)
+		)
+		(pin "1"
+		)
+		(pin "SH"
+		)
+		(pin "8"
+		)
+		(pin "7"
+		)
+		(pin "6"
+		)
+		(pin "5"
+		)
+		(pin "4"
+		)
+		(pin "3"
+		)
+		(pin "2"
+		)
+		(instances
+			(project "Kicad"
+				(path "/a972b0d3-46a0-4f09-b60b-5ab9fef2950e"
+					(reference "J3")
+					(unit 1)
+				)
