File: CAD/Kicad/Kicad.kicad_sch (KiCad schematic)
At the start: 72 parts, among them J1 USB_C_Receptacle_USB2.0_14P, J2 Conn_01x04_Pin, J3 RJ45_Shielded, J4 USB_C_Receptacle_USB2.0_14P, J5 USB_C_Receptacle_USB2.0_14P, J6 Conn_01x24_Pin, U1 ESP8266EX, U2 AMS1117, U3 SST25VF080B-50-4x-S2Ax, U4 FT230XS, U5 ESP32-S3-NEW, U6 FT230XS, U7 AMS1117, U8 SST25VF080B-50-4x-S2Ax, U9 AMS1117, Y1 Crystal_GND24, Y2 Crystal_GND23

Commit message: Journal entry and small PCB tweaks
Connections:
- net GND: no longer J3.1
- net MOSI: now reaches J3.7
- net MISO: now reaches J3.8
- new net MCLK: J3.1
Other:
- note added: "Add warning to NOT connect this to a non Cloudboard board or anything BUT the hubs/addons!"
- note removed: "Add warning to NOT connect this to a non Cloudboard board!"
Changed lines of the file:
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@@
 		)
 	)
-	(text "Add warning to NOT connect this to a non Cloudboard board!"
+	(text "Add warning to NOT connect this to a non Cloudboard board or anything BUT the hubs/addons!"
 		(exclude_from_sim no)
-		(at 79.248 202.438 0)
+		(at 90.17 200.406 0)
 		(effects
 			(font
@@
 	)
 	(junction
-		(at 33.02 231.14)
-		(diameter 0)
-		(color 0 0 0 0)
-	)
-	(junction
 		(at 177.8 186.69)
 		(diameter 0)
@@
 	)
 	(junction
-		(at 48.26 223.52)
-		(diameter 0)
-		(color 0 0 0 0)
-	)
-	(junction
 		(at 312.42 29.21)
 		(diameter 0)
@@
 	(wire
 		(pts
+			(xy 43.18 205.74) (xy 50.8 205.74)
+		)
+		(stroke
+			(width 0)
+			(type default)
+		)
+	)
+	(wire
+		(pts
 			(xy 270.51 153.67) (xy 274.32 153.67)
 		)
@@
 	(wire
 		(pts
-			(xy 33.02 231.14) (xy 33.02 245.11)
+			(xy 33.02 228.6) (xy 33.02 245.11)
 		)
 		(stroke
@@
 	(wire
 		(pts
-			(xy 48.26 231.14) (xy 48.26 223.52)
+			(xy 267.97 250.19) (xy 270.51 250.19)
 		)
 		(stroke
@@
 	(wire
 		(pts
-			(xy 267.97 250.19) (xy 270.51 250.19)
+			(xy 299.72 57.15) (xy 323.85 57.15)
 		)
 		(stroke
@@
 	(wire
 		(pts
-			(xy 299.72 57.15) (xy 323.85 57.15)
+			(xy 107.95 46.99) (xy 114.3 46.99)
 		)
 		(stroke
@@
 	(wire
 		(pts
-			(xy 107.95 46.99) (xy 114.3 46.99)
+			(xy 139.7 74.93) (xy 139.7 78.74)
 		)
 		(stroke
@@
 	(wire
 		(pts
-			(xy 139.7 74.93) (xy 139.7 78.74)
+			(xy 160.02 74.93) (xy 165.1 74.93)
 		)
 		(stroke
@@
 	(wire
 		(pts
-			(xy 160.02 74.93) (xy 165.1 74.93)
+			(xy 43.18 223.52) (xy 50.8 223.52)
 		)
 		(stroke
@@
 	(wire
 		(pts
-			(xy 43.18 223.52) (xy 48.26 223.52)
-		)
-		(stroke
-			(width 0)
-			(type default)
-		)
-	)
-	(wire
-		(pts
 			(xy 328.93 170.18) (xy 328.93 176.53)
 		)
@@
 	(wire
 		(pts
+			(xy 43.18 208.28) (xy 50.8 208.28)
+		)
+		(stroke
+			(width 0)
+			(type default)
+		)
+	)
+	(wire
+		(pts
 			(xy 175.26 20.32) (xy 175.26 17.78)
 		)
@@
 	(wire
 		(pts
-			(xy 48.26 223.52) (xy 50.8 223.52)
-		)
-		(stroke
-			(width 0)
-			(type default)
-		)
-	)
-	(wire
-		(pts
 			(xy 186.69 179.07) (xy 186.69 184.15)
 		)
@@
 	(wire
 		(pts
-			(xy 33.02 231.14) (xy 48.26 231.14)
-		)
-		(stroke
-			(width 0)
-			(type default)
-		)
-	)
-	(wire
-		(pts
 			(xy 193.04 118.11) (xy 199.39 118.11)
 		)
@@
 	(wire
 		(pts
-			(xy 33.02 231.14) (xy 33.02 228.6)
-		)
-		(stroke
-			(width 0)
-			(type default)
-		)
-	)
-	(wire
-		(pts
 			(xy 364.49 115.57) (xy 354.33 115.57)
 		)
@@
 		)
 	)
+	(label "MISO"
+		(at 50.8 205.74 0)
+		(effects
+			(font
+				(size 1.27 1.27)
+			)
+			(justify left bottom)
+		)
+	)
 	(label "MAIN_BUS_I2C_SDA"
 		(at 196.85 17.78 0)
@@
 		)
 	)
-	(label "I2C_COMMON_GND"
-		(at 50.8 223.52 0)
-		(effects
-			(font
-				(size 1.27 1.27)
-			)
-			(justify left bottom)
-		)
-	)
 	(label "ESP_8266_XIN"
 		(at 78.74 179.07 180)
@@
 		)
 	)
+	(label "MCLK"
+		(at 50.8 223.52 0)
+		(effects
+			(font
+				(size 1.27 1.27)
+			)
+			(justify left bottom)
+		)
+	)
 	(label "MAIN_BUS_I2C_SDA"
 		(at 287.02 121.92 180)
@@
 		(effects
 			(font
+				(size 1.27 1.27)
+			)
+			(justify left bottom)
+		)
+	)
+	(label "MOSI"
+		(at 50.8 208.28 0)
+		(effects
+			(font

Commit message: finished schematics and started PCB design
Parts:
- removed AE1, AE2: PCB_ANT, symbol Device:Antenna_Dipole
- removed C1, C12, C13, C14, C2, C24, C25: C, symbol Device:C
- removed C15, C16: 0.1uF, symbol Device:C
- removed C17, C20, C5, C6: 1uF, symbol Device:C
- removed C18: 10uF, symbol Device:C
- removed C19: 10nF, symbol Device:C
- removed C21, C22: 20pF, symbol Device:C
- removed C23: 100nF, symbol Device:C
- removed D1, D2, D6, D7: LED, symbol Device:LED
- removed D3: PWR_LED_1, symbol Device:LED
- removed D4: PWR_LED_2, symbol Device:LED
- removed D5: SD05C-01F, Diode_SMD:D_SOD-323, symbol Diode:SD05C-01F
- removed D8: PWR_LED_3, symbol Device:LED
- removed FB2, FB3: FerriteBead, symbol Device:FerriteBead
- removed J2: Conn_01x04_Pin, symbol Connector:Conn_01x04_Pin
- removed J3: RJ45_Shielded, symbol Connector:RJ45_Shielded
- removed J4, J5: USB_C_Receptacle_USB2.0_14P, symbol Connector:USB_C_Receptacle_USB2.0_14P
- removed J6: Conn_01x24_Pin, symbol Connector:Conn_01x24_Pin
- removed L1, L3, L4, L6: L, symbol Device:L
- removed L2: 4.3nH, symbol Device:L
- removed L5: 2.0nH, symbol Device:L
- removed R12K: 12K, symbol Device:R
- removed R_PWR_ADJ_1, R_PWR_ADJ_3, R_PWR_ADJ_5: 60, symbol Device:R
- removed R_PWR_ADJ_2, R_PWR_ADJ_4, R_PWR_ADJ_6: 100, symbol Device:R
- removed R_SPI_CLOCK: 200, symbol Device:R
- removed U1: ESP8266EX, Package_DFN_QFN:QFN-32-1EP_5x5mm_P0.5mm_EP3.45x3.45mm, symbol MCU_Espressif:ESP8266EX
- removed U2, U7, U9: AMS1117, Package_TO_SOT_SMD:SOT-223-3_TabPin2, symbol Regulator_Linear:AMS1117
- removed U3, U8: SST25VF080B-50-4x-S2Ax, Package_SO:SOIC-8_5.3x5.3mm_P1.27mm, symbol Memory_Flash:SST25VF080B-50-4x-S2Ax
- removed U4, U6: FT230XS, Package_SO:SSOP-16_3.9x4.9mm_P0.635mm, symbol Interface_USB:FT230XS
- removed U5: ESP32-S3-NEW, Package_DFN_QFN:QFN-56-1EP_7x7mm_P0.4mm_EP4x4mm, symbol New_Library:ESP32-S3-NEW
- removed Y1: Crystal_GND24, symbol Device:Crystal_GND24
- removed Y2: Crystal_GND23, symbol Device:Crystal_GND23
- added D1, D2: D_Schottky, Diode_SMD:D_SOD-123, symbol Device:D_Schottky
- added J2: USB_C_Receptacle_USB2.0_14P, Connector_USB:USB_C_Receptacle_Amphenol_12401610E4-2A, symbol Connector:USB_C_Receptacle_USB2.0_14P
- added J6: RJ45, Connector_RJ:RJ45_Amphenol_54602-x08_Horizontal, symbol Connector:RJ45
- added Q1, Q2: 2N3904, Package_TO_SOT_THT:TO-92_Inline, symbol Transistor_BJT:2N3904
- added R10, R11: 5K1, Resistor_SMD:R_0603_1608Metric_Pad0.98x0.95mm_HandSolder, symbol Device:R
- added R4, R5, R8: 12K, Resistor_SMD:R_0603_1608Metric_Pad0.98x0.95mm_HandSolder, symbol Device:R
- added R6: 12K, symbol Device:R
- added R7: 4.7K, Resistor_SMD:R_0603_1608Metric_Pad0.98x0.95mm_HandSolder, symbol Device:R
- added R9: 10K, symbol Device:R
- added SW1, SW2: SW_Push, Button_Switch_SMD:SW_SPST_EVQP2_MiddlePushTravel_H2.5mm, symbol Switch:SW_Push
- added U1: ESP32-S3-WROOM-2, RF_Module:ESP32-S3-WROOM-2, symbol RF_Module:ESP32-S3-WROOM-2
- added U3: AMS1117-3.3, Package_TO_SOT_SMD:SOT-223-3_TabPin2, symbol Regulator_Linear:AMS1117-3.3
- added U7: BME680, Package_LGA:Bosch_LGA-8_3x3mm_P0.8mm_ClockwisePinNumbering, symbol Sensor:BME680
- added U8: MPU-9250, Sensor_Motion:InvenSense_QFN-24_3x3mm_P0.4mm, symbol Sensor_Motion:MPU-9250
- added U9: FT231XQ, Package_DFN_QFN:QFN-20-1EP_4x4mm_P0.5mm_EP2.5x2.5mm, symbol Interface_USB:FT231XQ
- C10: value 100nF -> 0.1uF; footprint (none) -> Capacitor_SMD:C_0805_2012Metric
- C11, C9: value C -> 0.1uF; footprint (none) -> Capacitor_SMD:C_0805_2012Metric
- C3, C4: footprint (none) -> Capacitor_SMD:C_0805_2012Metric
- C7, C8: value 20pF -> 0.1uF; footprint (none) -> Capacitor_SMD:C_0805_2012Metric
- FB1: footprint (none) -> Inductor_SMD:L_0805_2012Metric_Pad1.05x1.20mm_HandSolder
- J1: footprint (none) -> Connector_USB:USB_C_Receptacle_Amphenol_12401610E4-2A
- R1: value 499 -> 5K1; footprint (none) -> Resistor_SMD:R_0603_1608Metric_Pad0.98x0.95mm_HandSolder
- R2: value 27K -> 5K1; footprint (none) -> Resistor_SMD:R_0603_1608Metric_Pad0.98x0.95mm_HandSolder
- R3: value 27K -> 10K
Connections:
- net ESP_8266_XOUT is gone; now on net VCC0: C8.1
- net MAIN_BUS_I2C_SCK is gone; now on net VCC0: R3.1
- net MAIN_BUS_I2C_SDA is gone; now on an unnamed net: R2.1
- net MPU_U0TXD is gone; now on net GND: R1.2
- net GND: now also C4.2, J1.A1 (GND), J1.A12 (GND), J1.B1 (GND), J1.B12 (GND), J1.SH (SHIELD), R2.2, J2.A1 (GND), J2.A12 (GND), J2.B1 (GND), J2.B12 (GND), J2.SH (SHIELD), J6.5, R10.2, R11.2, R4.2, R8.1, U1.1 (GND), U1.40 (GND), U1.41 (GND), U3.1 (GND), U7.1 (GND), U7.7 (GND), U8.18 (GND), U8.20 (RESV_GND), U9.13 (GND), U9.21 (GND), U9.3 (GND); no longer C3.1, C4.1, C7.1, C8.2, C9.2, FB1.2
- net VCC0: now also C3.1, C7.1, C9.1, J6.6, R7.2, R9.1, U3.2 (VO), U8.1 (RESV_VDDIO), U9.12 (VCC); no longer C3.2, C4.2
- net at C11.1: now also U8.10 (REGOUT)
- net at J1.A5 (CC1): now also R1.1
- net ESP32_AUTORST: now reaches R3.2
- net ESP32_AUTORST: now also Q2.3 (C), SW1.2, U1.3 (EN)
- net A_5V renamed 5V_USB_0
- net 5V_USB_0: now also FB1.1, D2.2 (A); no longer C9.1
- net ESP_8266_USB_D+ renamed SERIAL_D+
- net SERIAL_D+: now also U9.8 (USBDP)
- net ESP_8266_USB_D- renamed SERIAL_D-
- net SERIAL_D-: now also U9.9 (USBDM)
- net ESP_8266_XIN: no longer names the net of C7.2
- net ESP_8266_XIN: now also U7.8 (VDD)
- net ZRI_U0TXD: no longer names the net of C10.2
- net ZRI_U0TXD: now also U8.8 (VDDIO)
- new net: C9.2, U8.13 (VDD)
- new net: R8.2, SW2.2
- new net: Q1.2 (B), R6.2
- new net: R4.1, SW1.1
- new net: C3.2, U1.2 (3V3)
- new net: J2.B5 (CC2), R11.1
- new net: C8.2, U7.6 (VDDIO)
- new net: FB1.2, J2.A4 (VBUS), J2.A9 (VBUS), J2.B4 (VBUS), J2.B9 (VBUS)
- new net: Q2.2 (B), R5.2
- new net: J2.A5 (CC1), R10.1
- new net BOOT: Q1.3 (C), R7.1, R9.2, SW2.1, U1.27 (IO0)
- new net CBUS0: U9.15 (CBUS0)
- new net CBUS1: U9.14 (CBUS1)
- new net CS_BUS_A: J6.1, U1.18 (IO10)
- new net CS_BUS_B: U7.2 (CSB), U8.22 (~{CS})
- new net DTR_A: Q1.1 (E), R5.1, U9.18 (~{DTR})
- new net ESP32_RXD: U1.36 (RXD0/IO44), U9.17 (TXD)
- new net ESP32_S3_IO0: U8.12 (INT)
- new net ESP32_TXD: U1.37 (TXD0/IO43), U9.1 (RXD)
- new net IO1: U1.39 (IO1)
- new net IO14: U1.22 (IO14)
- new net IO15: U1.8 (IO15)
- new net IO16: U1.9 (IO16)
- new net IO17: U1.10 (IO17)
- new net IO18: U1.11 (IO18)
- new net IO2: U1.38 (IO2)
- new net IO21: U1.23 (IO21)
- new net IO3: U1.15 (IO3)
- new net IO38: U1.31 (IO38)
- new net IO39: U1.32 (MTCK/IO39)
- new net IO4: U1.4 (IO4)
- new net IO40: U1.33 (MTDO/IO40)
- new net IO41: U1.34 (MTDI/IO41)
- new net IO42: U1.35 (MTMS/IO42)
- new net IO45: U1.26 (IO45)
- new net IO46: U1.16 (IO46)
- new net IO47: U1.24 (IO47)
- new net IO48: U1.25 (IO48)
- new net IO5: U1.5 (IO5)
- new net IO6: U1.6 (IO6)
- new net IO7: U1.7 (IO7)
- new net IO8: U1.12 (IO8)
- new net IO9: U1.17 (IO9)
- new net IOOUT_A: C4.1, U9.10 (3V3OUT), U9.11 (~{RESET}), U9.20 (VCCIO)
- new net MISO_BUS_A: J6.2, U1.21 (IO13)
- new net MISO_BUS_B: U7.3 (SDI), U8.9 (AD0/MISO)
- new net MOSI_BUS_A: J6.4, U1.19 (IO11)
- new net MOSI_BUS_B: U7.5 (SDO), U8.24 (SDA/MOSI)
- new net NATIVE_D+: J2.A6 (D+), J2.B6 (D+), U1.14 (USB_D+/IO20)
- new net NATIVE_D-: J2.A7 (D-), J2.B7 (D-), U1.13 (USB_D-/IO19)
- new net OROUT: D1.1 (K), D2.1 (K), U3.3 (VI)
- new net RJ43_P7: J6.7
- new net RJ43_P8: J6.8
- new net RTS_A: Q2.1 (E), R6.1, U9.19 (~{RTS})
- new net SCK_BUS_A: J6.3
- new net SCK_BUS_B: U7.4 (SCK), U8.23 (SCL/SCLK)
- new net SPICLK_BUS_A: U1.20 (IO12)
- new net VIN: D1.2 (A)
- no-connect marks 0 -> 3
Other:
- note added: "Auto reset"
- note removed: "(Matching of Antenna)"
- note removed: "(Matching of Chip)"
- note removed: "40 MhZ +- 10PPM"
- note removed: "40MhZ +- 10 PPM"
- note removed: "Add R1 if needed"
- note removed: "Add warning to NOT connect this to a non Cloudboard board or anything BUT the hubs/addons!"
- note removed: "All varibles past LNA_IN are TBD"
- note removed: "Crystal Circuit To Drive ZRI"
- note removed: "Crystal Unit for ESP32-S3"
- note removed: "Database and hub connections will be initialized through I2C VIA GPIO pins 8 carrying data and 9 carrying clock"
- note removed: "ESP-S3 ANT"
- note removed: "ESP8266 Zero Ring Interface Unit (ZRI)"
- note removed: "External plugs to power both MCU units and sensing board [5V ONLY!!!]"
- note removed: "I2C Pull up"
- note removed: "I2C Serial connection to join both MCUs"
- note removed: "MPU Direct USB Port"
- note removed: "MPU Power Supply"
- note removed: "MPU UART USB Port"
- note removed: "MPU USB to UART IC"
- note removed: "Maybe find a better way to carry I2C..."
- note removed: "RJ45 sensor board connector"
- note removed: "Sensor 3v3 supply"
- note removed: "Single-ended 50 ohm RF traces"
- note removed: "Soon to be GPIO headers"
- note removed: "USB to UART IC"
- note removed: "Values of L1, C1, and C2 are soon to be found"
- note removed: "Values subject to change"
- note removed: "ZRI Flash"
- note removed: "ZRI Power Supply"
- note removed: "ZRI USB Port"
- title: Cloudboard Processing Main Unit -> (none)

Commit message: started PCB
Parts:
- added FB2: FerriteBead, Inductor_SMD:L_0805_2012Metric_Pad1.05x1.20mm_HandSolder, symbol Device:FerriteBead
- added J3, J4: Conn_01x20_Pin, Connector_PinHeader_2.54mm:PinHeader_1x20_P2.54mm_Vertical, symbol Connector:Conn_01x20_Pin
- Q1, Q2: footprint Package_TO_SOT_THT:TO-92_Inline -> Package_TO_SOT_THT:TO-92S
- R3, R6, R9: footprint (none) -> Resistor_SMD:R_0603_1608Metric_Pad0.98x0.95mm_HandSolder
Connections:
- net 5V_USB_0: no longer J1.A4 (VBUS), J1.A9 (VBUS), J1.B4 (VBUS), J1.B9 (VBUS)
- net BOOT: now also J4.7 (Pin_7)
- net CS_BUS_A: now also U7.2 (CSB), J4.17 (Pin_17)
- net CS_BUS_B: no longer U7.2 (CSB)
- net ESP32_RXD: now also J3.15 (Pin_15)
- net ESP32_TXD: now also J3.14 (Pin_14)
- net GND: now also J4.2 (Pin_2), J4.3 (Pin_3)
- net IO1: now also J4.8 (Pin_8)
- net IO14: now also J3.1 (Pin_1)
- net IO15: now also J3.2 (Pin_2)
- net IO16: now also J3.3 (Pin_3)
- net IO17: now also J3.4 (Pin_4)
- net IO18: now also J3.5 (Pin_5)
- net IO2: now also J4.9 (Pin_9)
- net IO21: now also J3.8 (Pin_8)
- net IO3: now also J4.10 (Pin_10)
- net IO38: now also J3.9 (Pin_9)
- net IO39: now also J3.10 (Pin_10)
- net IO4: now also J4.11 (Pin_11)
- net IO40: now also J3.11 (Pin_11)
- net IO41: now also J3.12 (Pin_12)
- net IO42: now also J3.13 (Pin_13)
- net IO45: now also J3.16 (Pin_16)
- net IO46: now also J3.17 (Pin_17)
- net IO47: now also J3.18 (Pin_18)
- net IO48: now also J3.19 (Pin_19)
- net IO5: now also J4.12 (Pin_12)
- net IO6: now also J4.13 (Pin_13)
- net IO7: now also J4.14 (Pin_14)
- net IO8: now also J4.15 (Pin_15)
- net IO9: now also J4.16 (Pin_16)
- net MISO_BUS_A: now also U7.3 (SDI), J4.20 (Pin_20)
- net MISO_BUS_B: no longer U7.3 (SDI)
- net MOSI_BUS_A: now also U7.5 (SDO), J4.18 (Pin_18)
- net MOSI_BUS_B: no longer U7.5 (SDO)
- net NATIVE_D+: now also J3.7 (Pin_7)
- net NATIVE_D-: now also J3.6 (Pin_6)
- net OROUT: now also J4.1 (Pin_1)
- net RJ43_P7: now also J4.6 (Pin_6)
- net RJ43_P8: now also J4.5 (Pin_5)
- net SCK_BUS_A: now also U7.4 (SCK)
- net SCK_BUS_B: no longer U7.4 (SCK)
- net SPICLK_BUS_A: now also J4.19 (Pin_19)
- net VCC0: now also J4.4 (Pin_4)
- net VIN: now also J3.20 (Pin_20)
- net ESP32_S3_IO0: no longer names the net of U8.12 (INT)
- new net: FB2.2, J1.A4 (VBUS), J1.A9 (VBUS), J1.B4 (VBUS), J1.B9 (VBUS)
- new net 5V_USB_1: FB2.1

Commit message: PCB work and journal entry
Parts:
- added D3, D4: D_Schottky, Diode_SMD:D_SOD-123, symbol Device:D_Schottky
Connections:
- net CS_BUS_B is gone; now on net CS_BUS_A: U8.22 (~{CS})
- net MISO_BUS_B is gone; now on net MISO_BUS_A: U8.9 (AD0/MISO)
- net MOSI_BUS_B is gone; now on net MOSI_BUS_A: U8.24 (SDA/MOSI)
- net SCK_BUS_B is gone; now on net SCK_BUS_A: U8.23 (SCL/SCLK)
- net SPICLK_BUS_A is gone; now on net SCK_BUS_A: J4.19 (Pin_19), U1.20 (IO12)
- net 5V_USB_0: now also FB1.2, J2.A4 (VBUS), J2.A9 (VBUS), J2.B4 (VBUS), J2.B9 (VBUS), D3.2 (A); no longer D2.2 (A)
- net 5V_USB_1: now also FB2.2, J1.A4 (VBUS), J1.A9 (VBUS), J1.B4 (VBUS), J1.B9 (VBUS), D4.2 (A)
- net VCC0: now also C3.2, U1.2 (3V3)
- new net: D2.2 (A), D3.1 (K), D4.1 (K)

Commit message: Finalized PCB (Yes!)
Connections:
- net CBUS0: no longer U9.15 (CBUS0)
- net CBUS1: no longer U9.14 (CBUS1)
- no-connect marks 3 -> 12
Other:
- title: (none) -> Cloudboard Low Power Module Final Schematic
Changed lines of the file:
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@@
 	(generator_version "10.0")
 	(paper "A4")
+	(title_block
+		(title "Cloudboard Low Power Module Final Schematic")
+		(date "2026-05-18")
+		(rev "2")
+		(comment 1 "Matias Argandoña")
+		(comment 2 "C 2026")
+	)
 	(text "Auto reset\n"
 		(exclude_from_sim no)
@@
 	)
 	(no_connect
+		(at 200.66 140.97)
+	)
+	(no_connect
 		(at 270.51 128.27)
+	)
+	(no_connect
+		(at 199.39 138.43)
+	)
+	(no_connect
+		(at 200.66 130.81)
+	)
+	(no_connect
+		(at 200.66 133.35)
+	)
+	(no_connect
+		(at 200.66 143.51)
+	)
+	(no_connect
+		(at 200.66 138.43)
+	)
+	(no_connect
+		(at 200.66 128.27)
+	)
+	(no_connect
+		(at 200.66 146.05)
 	)
 	(no_connect
@@
 	(no_connect
 		(at 270.51 130.81)
+	)
+	(no_connect
+		(at 200.66 123.19)
 	)
 	(wire
@@
 	)
 	(label "CBUS1"
-		(at 200.66 140.97 0)
+		(at 207.01 140.97 0)
 		(fields_autoplaced yes)
 		(effects
@@
 		)
 		(property "Net Class" "I/O"
-			(at 200.66 142.24 0)
+			(at 207.01 142.24 0)
 			(show_name no)
 			(do_not_autoplace no)
@@
 	)
 	(label "CBUS0"
-		(at 200.66 138.43 0)
+		(at 207.01 138.43 0)
 		(fields_autoplaced yes)
 		(effects
@@
 		)
 		(property "Net Class" "I/O"
-			(at 200.66 139.7 0)
+			(at 207.01 139.7 0)
 			(show_name no)
 			(do_not_autoplace no)

Commit message: finished then scrapped rev1
Parts:
- removed J6: RJ45, Connector_RJ:RJ45_Amphenol_54602-x08_Horizontal, symbol Connector:RJ45
Connections:
- net IOOUT_A is gone; now on net VCC0: C4.1, U9.10 (3V3OUT), U9.11 (~{RESET}), U9.20 (VCCIO)
- net RJ43_P7 is gone; now on net VCC0: J4.6 (Pin_6)
- net RJ43_P8 is gone; now on net OROUT: J4.5 (Pin_5)
- net GND: no longer R2.2
- net NATIVE_D+: no longer J3.7 (Pin_7)
- net NATIVE_D-: no longer J3.6 (Pin_6)
Other:
- note added: "ESP32-S3"
- note added: "Env sensor"
- note added: "GPIO Header"
- note added: "IMU IC"
- note added: "Power ORing"
- note added: "Serial USB"
- note added: "Serial USB port"
- note added: "USB to Serial IC"
- note added: "Voltage Regulator"
- title: Cloudboard Low Power Module Final Schematic -> S3 Low Power Devboard
- moved on the sheet: C3, C4, FB1, J2, J3, Q1, Q2, R10, R11, R3, R4, R5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
