File: CAD/Kicad/Kicad.kicad_pcb (KiCad board)
At the start: 2 copper layers, 31 parts, among them J1 USB_C_Receptacle_USB2.0_14P, J2 USB_C_Receptacle_USB2.0_14P, J3 Conn_01x33_Pin, J6 RJ45, Q1 2N3904, Q2 2N3904, SW1 SW_Push, SW2 SW_Push, U1 ESP32-S3-WROOM-2, U3 AMS1117-3.3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

Commit message: started PCB
Parts:
- added FB2: FerriteBead, Inductor_SMD:L_0805_2012Metric_Pad1.05x1.20mm_HandSolder, F.Cu at (237.3, 103.0)
- added J4: Conn_01x20_Pin, Connector_PinHeader_2.54mm:PinHeader_1x20_P2.54mm_Vertical, F.Cu at (183.4, 69.8)
- J3: value Conn_01x33_Pin -> Conn_01x20_Pin; footprint Connector_PinSocket_2.54mm:PinSocket_1x33_P2.54mm_Vertical_SMD_Pin1Left -> Connector_PinHeader_2.54mm:PinHeader_1x20_P2.54mm_Vertical
- moved R8 104.8 mm to (254.0, 88.1), turned to 90 degrees
- moved R5 98.3 mm to (249.0, 88.1), turned to 90 degrees
- moved C11 97.5 mm to (238.7, 88.0), turned to 90 degrees
- moved R4 95.0 mm to (246.5, 88.1), turned to 90 degrees
- moved C10 93.5 mm to (235.7, 88.0), turned to 90 degrees
- moved R2 91.8 mm to (244.0, 88.1), turned to 90 degrees
- moved C9 89.4 mm to (232.7, 88.0), turned to 90 degrees
- moved R1 88.6 mm to (241.4, 88.1), turned to 90 degrees
- moved J6 87.1 mm to (251.3, 124.7)
- moved C8 85.4 mm to (229.7, 88.0), turned to 90 degrees
- moved R7 85.3 mm to (237.0, 95.5), turned to 90 degrees
- moved R11 83.9 mm to (241.0, 125.1), turned to -90 degrees
- moved C7 81.3 mm to (226.7, 88.0), turned to 90 degrees
- moved R10 77.7 mm to (235.0, 125.0), turned to 90 degrees
- moved C4 77.3 mm to (223.6, 88.0), turned to 90 degrees
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Connections:
- J1 pad A4: /5V_USB_0 -> Net-(FB2-Pad2)
- J1 pad A9: /5V_USB_0 -> Net-(FB2-Pad2)
- J1 pad B4: /5V_USB_0 -> Net-(FB2-Pad2)
- J1 pad B9: /5V_USB_0 -> Net-(FB2-Pad2)
- J3 pad 1: /BOOT -> /IO14
- J3 pad 10: /IO9 -> /IO39
- J3 pad 11: /CS_BUS_A -> /IO40
- J3 pad 12: /MOSI_BUS_A -> /IO41
- J3 pad 13: /SPICLK_BUS_A -> /IO42
- J3 pad 14: /MISO_BUS_A -> /ESP32_TXD
- J3 pad 15: /IO14 -> /ESP32_RXD
- J3 pad 16: /IO15 -> /IO45
- J3 pad 17: /IO16 -> /IO46
- J3 pad 18: /IO17 -> /IO47
- J3 pad 19: /IO18 -> /IO48
- J3 pad 2: /IO1 -> /IO15
- J3 pad 20: /NATIVE_D- -> /VIN
- J3 pad 3: /IO2 -> /IO16
- J3 pad 4: /IO3 -> /IO17
- J3 pad 5: /IO4 -> /IO18
- J3 pad 6: /IO5 -> /NATIVE_D-
- J3 pad 7: /IO6 -> /NATIVE_D+
- J3 pad 8: /IO7 -> /IO21
- J3 pad 9: /IO8 -> /IO38
- J6 pad 2: /VCC0 -> /MISO_BUS_A
- J6 pad 3: /MISO_BUS_A -> /SCK_BUS_A
- J6 pad 4: /GND -> /MOSI_BUS_A
- J6 pad 5: /SCK_BUS_A -> /GND
- J6 pad 6: unconnected-(J6-Pad6) -> /VCC0
- J6 pad 7: /MOSI_BUS_A -> /RJ43_P7
- J6 pad 8: unconnected-(J6-Pad8) -> /RJ43_P8
- U7 pad 2: /CS_BUS_B -> /CS_BUS_A
- U7 pad 3: /MISO_BUS_B -> /MISO_BUS_A
- U7 pad 4: /SCK_BUS_B -> /SCK_BUS_A
- U7 pad 5: /MOSI_BUS_B -> /MOSI_BUS_A
- U8 pad 12: /ESP32_S3_IO0 -> unconnected-(U8-INT-Pad12)
- U9 pad 14: unconnected-(U9-CBUS1-Pad14) -> /CBUS1
- U9 pad 15: unconnected-(U9-CBUS0-Pad15) -> /CBUS0
Routing:
- net /NATIVE_D+: track 0.00 -> 82.3 mm
- net /NATIVE_D-: track 0.00 -> 71.1 mm
- net /GND: track 0.00 -> 26.1 mm
- net Net-(J2-CC2): track 0.00 -> 16.3 mm
- net Net-(J2-CC1): track 0.00 -> 5.20 mm
- net Net-(FB1-Pad2): track 0.00 -> 1.80 mm
- net (no net): vias 0 -> 1
Other:
- board outline added: 50.5 x 100 mm

Commit message: PCB work and journal entry
Parts:
- added D3: D_Schottky, Diode_SMD:D_SOD-123, F.Cu at (186.5, 75.8)
- added D4: D_Schottky, Diode_SMD:D_SOD-123, F.Cu at (178.0, 70.0)
- added R3: 10K, Resistor_SMD:R_0603_1608Metric_Pad0.98x0.95mm_HandSolder, F.Cu at (182.0, 64.5)
- added R6: 12K, Resistor_SMD:R_0603_1608Metric_Pad0.98x0.95mm_HandSolder, F.Cu at (213.0, 77.5)
- added R9: 10K, Resistor_SMD:R_0603_1608Metric_Pad0.98x0.95mm_HandSolder, F.Cu at (212.0, 65.5)
- Q1, Q2: footprint Package_TO_SOT_THT:TO-92_Inline -> Package_TO_SOT_THT:TO-92S
- moved J6 91.2 mm to (172.3, 79.2)
- moved C8 67.5 mm to (170.0, 56.5), turned to -90 degrees
- moved J2 65.1 mm to (193.0, 87.7)
- moved R10 65.0 mm to (189.6, 78.5), turned to 180 degrees
- moved D1 62.5 mm to (172.8, 68.0)
- moved C7 62.3 mm to (173.5, 55.5), turned to -90 degrees
- moved D2 62.0 mm to (172.8, 72.5)
- moved FB1 61.4 mm to (187.8, 80.5)
- moved FB2 61.2 mm to (184.0, 73.0), turned to 90 degrees
- moved U3 60.9 mm to (219.3, 58.5)
- moved J3 60.9 mm to (230.0, 36.9)
- moved R11 60.2 mm to (200.0, 81.0), turned to 0 degrees
- moved U7 53.0 mm to (172.8, 59.7)
- moved C3 50.0 mm to (181.1, 57.5), turned to 0 degrees
- moved Q2 50.0 mm to (204.7, 74.4)
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Connections:
- C3 pad 2: Net-(U1-3V3) -> /VCC0
- D2 pad 2: /5V_USB_0 -> Net-(D2-A)
- FB1 pad 2: Net-(FB1-Pad2) -> /5V_USB_0
- FB2 pad 2: Net-(FB2-Pad2) -> /5V_USB_1
- J1 pad A4: Net-(FB2-Pad2) -> /5V_USB_1
- J1 pad A9: Net-(FB2-Pad2) -> /5V_USB_1
- J1 pad B4: Net-(FB2-Pad2) -> /5V_USB_1
- J1 pad B9: Net-(FB2-Pad2) -> /5V_USB_1
- J2 pad A4: Net-(FB1-Pad2) -> /5V_USB_0
- J2 pad A9: Net-(FB1-Pad2) -> /5V_USB_0
- J2 pad B4: Net-(FB1-Pad2) -> /5V_USB_0
- J2 pad B9: Net-(FB1-Pad2) -> /5V_USB_0
- J4 pad 19: /SPICLK_BUS_A -> /SCK_BUS_A
- U1 pad 2: Net-(U1-3V3) -> /VCC0
- U1 pad 20: /SPICLK_BUS_A -> /SCK_BUS_A
- U8 pad 22: /CS_BUS_B -> /CS_BUS_A
- U8 pad 23: /SCK_BUS_B -> /SCK_BUS_A
- U8 pad 24: /MOSI_BUS_B -> /MOSI_BUS_A
- U8 pad 9: /MISO_BUS_B -> /MISO_BUS_A
Routing:
- net /MISO_BUS_A: track 0.00 -> 213.9 mm, vias 0 -> 4
- net /GND: track 26.1 -> 216.8 mm, vias 0 -> 6
- net /SCK_BUS_A: track 0.00 -> 147.1 mm, vias 0 -> 5
- net /CS_BUS_A: track 0.00 -> 137.9 mm, vias 0 -> 7
- net /IO9: track 0.00 -> 136.3 mm, vias 0 -> 5
- net /MOSI_BUS_A: track 0.00 -> 126.9 mm, vias 0 -> 4
- net /IO7: track 0.00 -> 116.4 mm, vias 0 -> 2
- net /IO6: track 0.00 -> 114.5 mm, vias 0 -> 2
- net /IO3: track 0.00 -> 113.8 mm, vias 0 -> 1
- net /IO5: track 0.00 -> 112.3 mm, vias 0 -> 1
- net /ESP32_AUTORST: track 0.00 -> 106.2 mm, vias 0 -> 1
- net /OROUT: track 0.00 -> 97.1 mm, vias 0 -> 4
- net /VCC0: track 0.00 -> 86.9 mm, vias 0 -> 8
- net /IO2: track 0.00 -> 84.8 mm, vias 0 -> 1
- net /BOOT: track 0.00 -> 71.3 mm, vias 0 -> 1
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- added copper zone on In2.Cu, net /VCC0
Other:
- board size 50.5 x 100 mm -> 69.5 x 63 mm
- copper layers 2 -> 6
- board text added: "BOOT"
- board text added: "EN"

Commit message: Finalized PCB (Yes!)
Parts:
- moved J3 105.0 mm to (125.0, 34.8)
- moved SW1 96.9 mm to (138.9, 45.1), turned to 0 degrees
- moved R4 89.2 mm to (143.1, 41.0), turned to 0 degrees
- moved SW2 86.4 mm to (137.9, 55.1), turned to 0 degrees
- moved R8 82.0 mm to (138.9, 59.5), turned to 0 degrees
- moved C9 57.8 mm to (162.5, 62.0), turned to 0 degrees
- moved J1 54.0 mm to (153.5, 80.5)
- moved R2 53.5 mm to (159.5, 64.5), turned to 90 degrees
- moved C10 50.0 mm to (166.1, 60.5)
- moved C4 50.0 mm to (152.5, 61.0)
- moved U8 49.4 mm to (170.5, 63.0)
- moved R1 48.4 mm to (157.1, 68.5), turned to 90 degrees
- moved C11 48.2 mm to (175.0, 62.5), turned to 0 degrees
- moved R6 47.6 mm to (166.6, 67.0), turned to 0 degrees
- moved R7 46.7 mm to (176.0, 54.5), turned to 90 degrees
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Connections:
- U9 pad 14: /CBUS1 -> unconnected-(U9-CBUS1-Pad14)
- U9 pad 15: /CBUS0 -> unconnected-(U9-CBUS0-Pad15)
Routing:
- net /VCC0: track 86.9 -> 200.9 mm, vias 8 -> 3
- net /RJ43_P8: track 41.6 -> 144.0 mm
- net /GND: track 216.8 -> 316.6 mm
- net /IO9: track 136.3 -> 36.8 mm, vias 5 -> 1
- net /NATIVE_D-: track 29.5 -> 128.5 mm, vias 2 -> 3
- net /IO3: track 113.8 -> 27.2 mm
- net /IO7: track 116.4 -> 33.4 mm, vias 2 -> 1
- net /MISO_BUS_A: track 213.9 -> 134.0 mm, vias 4 -> 2
- net /NATIVE_D+: track 29.2 -> 102.5 mm, vias 3 -> 4
- net /IO48: track 0.00 -> 73.0 mm, vias 0 -> 1
- net /IO47: track 0.00 -> 69.5 mm, vias 0 -> 1
- net /IO42: track 0.00 -> 64.9 mm, vias 0 -> 1
- net /IO41: track 0.00 -> 62.7 mm, vias 0 -> 1
- net /IO40: track 0.00 -> 61.3 mm, vias 0 -> 1
- net /IO39: track 0.00 -> 60.3 mm, vias 0 -> 1
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- removed copper zone on In2.Cu, net /VCC0
Other:
- board size 69.5 x 63 mm -> 72.5 x 53 mm
- board text added: "Designed by:"
- board text added: "Matias Argandona"
- board text added: "Put that back =("
- board text added: "Rev 1 PROTOTYPE"

Commit message: finished then scrapped rev1
Parts:
- removed J6: RJ45, Connector_RJ:RJ45_Amphenol_54602-x08_Horizontal
- moved J3 96.5 mm to (214.0, 72.0)
- moved R9 96.1 mm to (84.5, 75.3), turned to 0 degrees
- moved R7 92.8 mm to (84.5, 70.3), turned to 0 degrees
- moved R11 91.1 mm to (84.5, 80.3)
- moved SW1 89.5 mm to (65.4, 96.2)
- moved C11 88.1 mm to (88.5, 46.1)
- moved R10 88.1 mm to (84.5, 77.8), turned to 0 degrees
- moved J4 87.8 mm to (210.0, 72.0)
- moved R3 79.9 mm to (80.2, 75.3), turned to 0 degrees
- moved R2 79.7 mm to (80.2, 72.8), turned to 0 degrees
- moved C10 79.5 mm to (88.5, 43.1)
- moved C9 77.2 mm to (88.5, 40.0)
- moved R1 76.9 mm to (80.2, 70.3), turned to 0 degrees
- moved C7 76.7 mm to (195.0, 105.5)
- moved D1 76.5 mm to (203.7, 107.0)
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Connections:
- C11 pad 2: /GND -> GND
- C4 pad 1: /IOOUT_A -> /VCC0
- C4 pad 2: /GND -> GND
- J1 pad A1: /GND -> GND
- J1 pad A12: /GND -> GND
- J1 pad B1: /GND -> GND
- J1 pad B12: /GND -> GND
- J1 pad SH: /GND -> GND
- J2 pad A1: /GND -> GND
- J2 pad A12: /GND -> GND
- J2 pad B1: /GND -> GND
- J2 pad B12: /GND -> GND
- J2 pad SH: /GND -> GND
- J3 pad 6: /NATIVE_D- -> unconnected-(J3-Pin_6-Pad6)
- J3 pad 7: /NATIVE_D+ -> unconnected-(J3-Pin_7-Pad7)
- J4 pad 2: /GND -> GND
- J4 pad 3: /GND -> GND
- J4 pad 5: /RJ43_P8 -> /OROUT
- J4 pad 6: /RJ43_P7 -> /VCC0
- R1 pad 2: /GND -> GND
- R10 pad 2: /GND -> GND
- R11 pad 2: /GND -> GND
- R2 pad 2: /GND -> unconnected-(R2-Pad2)
- R4 pad 2: /GND -> GND
- R8 pad 1: /GND -> GND
- U1 pad 1: /GND -> GND
- U1 pad 40: /GND -> GND
- U1 pad 41: /GND -> GND
- U3 pad 1: /GND -> GND
- U7 pad 1: /GND -> GND
- U7 pad 7: /GND -> GND
- U8 pad 18: /GND -> GND
- U8 pad 20: /GND -> GND
- U9 pad 10: /IOOUT_A -> /VCC0
- U9 pad 11: /IOOUT_A -> /VCC0
- U9 pad 13: /GND -> GND
- U9 pad 20: /IOOUT_A -> /VCC0
- U9 pad 21: /GND -> GND
- U9 pad 3: /GND -> GND
Routing:
- net /GND: track 316.6 -> 0.00 mm, vias 6 -> 0
- net /VCC0: track 200.9 -> 37.2 mm, vias 3 -> 0
- net GND: track 0.00 -> 148.3 mm, vias 0 -> 2
- net /RJ43_P8: track 144.0 -> 0.00 mm
- net /CS_BUS_A: track 150.9 -> 14.7 mm
- net /NATIVE_D-: track 128.5 -> 0.00 mm, vias 3 -> 0
- net /SCK_BUS_A: track 132.9 -> 10.5 mm, vias 3 -> 0
- net /MISO_BUS_A: track 134.0 -> 12.8 mm, vias 2 -> 0
- net /BOOT: track 117.1 -> 0.00 mm, vias 3 -> 0
- net /NATIVE_D+: track 102.5 -> 0.00 mm, vias 4 -> 0
- net /ESP32_TXD: track 90.2 -> 0.00 mm, vias 1 -> 0
- net /IO2: track 89.6 -> 0.00 mm, vias 1 -> 0
- net /RJ43_P7: track 85.4 -> 0.00 mm
- net /OROUT: track 108.0 -> 23.9 mm, vias 1 -> 0
- net /ESP32_AUTORST: track 83.8 -> 0.00 mm, vias 2 -> 0
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Other:
- board size 72.5 x 53 mm -> 33 x 61 mm
- copper layers 6 -> 2
- board text removed: "BOOT"
- board text removed: "Designed by:"
- board text removed: "EN"
- board text removed: "Matias Argandona"
- board text removed: "Put that back =("
- board text removed: "Rev 1 PROTOTYPE"
